File: prova-buck.kicad_sch (KiCad schematic)
At the start: 44 parts, among them J1 Screw_Terminal_01x02, J2 Barrel_Jack_MountingPin, J3 USB_B_Micro, J4 Conn_02x03_Odd_Even, J5 Conn_02x03_Odd_Even, J6 Conn_01x04, J7 Conn_01x04, J8 Conn_01x02, J9 Conn_01x02, Q1 AO3401A, Q2 AO3401A, U1 MPQ9842GL, U2 LDL1117S33R, U3 LM358

Commit message: Generated BOM adn CPL file
Parts:
- C1, C2: LCSC Part (none) -> C13585
- C10, C11: LCSC Part (none) -> C12891
- C12: LCSC Part (none) -> C23630
- C13: LCSC Part (none) -> C1779
- C3: LCSC Part (none) -> C15849
- C4, C5, C7: LCSC Part (none) -> C14663
- C6: LCSC Part (none) -> C307331
- C8: LCSC Part (none) -> C19666
- C9: LCSC Part (none) -> C1634
- D1: LCSC Part (none) -> C8678
- D2, D4, F1, J1, J2, J3, J4, J5, J6, J7, J8, J9, U1, U2: JLCPCB BOM (none) -> 0
- D3: LCSC Part (none) -> C72041
- L1: LCSC Part (none) -> C408412
- Q1, Q2: LCSC Part (none) -> C15127
- R1, R2: LCSC Part (none) -> C25803
- R10: LCSC Part (none) -> C31850
- R11: LCSC Part (none) -> C23253
- R3: LCSC Part (none) -> C23254
- R4: LCSC Part (none) -> C23231
- R5: LCSC Part (none) -> C22797
- R6: LCSC Part (none) -> C22859
- R7: LCSC Part (none) -> C25819
- R8: LCSC Part (none) -> C25077
- R9: LCSC Part (none) -> C23189
- U3: LCSC Part (none) -> C7950
Changed lines of the file:
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@@
+      (effects (font (size 1.27 1.27)) hide)
+    )
+    (property "LCSC Part" "C25803" (id 5) (at 104.14 64.77 0)
       (effects (font (size 1.27 1.27)) hide)
     )
@@
       (effects (font (size 1.27 1.27)) hide)
     )
+    (property "LCSC Part" "C13585" (id 5) (at 113.03 36.83 0)
+      (effects (font (size 1.27 1.27)) hide)
+    )
     (pin "1")
     (pin "2")
@@
     )
     (property "Datasheet" "~" (id 3) (at 25.4 76.2 0)
+      (effects (font (size 1.27 1.27)) hide)
+    )
+    (property "JLCPCB BOM" "0" (id 4) (at 25.4 76.2 0)
       (effects (font (size 1.27 1.27)) hide)
     )
@@
       (effects (font (size 1.27 1.27)) hide)
     )
+    (property "LCSC Part" "C13585" (id 5) (at 120.65 36.83 0)
+      (effects (font (size 1.27 1.27)) hide)
+    )
     (pin "1")
     (pin "2")
@@
       (effects (font (size 1.27 1.27)) hide)
     )
+    (property "LCSC Part" "C14663" (id 5) (at 128.27 36.83 0)
+      (effects (font (size 1.27 1.27)) hide)
+    )
     (pin "1")
     (pin "2")
@@
     )
     (property "LCSC Part #" "C14663" (id 4) (at 135.89 36.83 0)
+      (effects (font (size 1.27 1.27)) hide)
+    )
+    (property "LCSC Part" "C14663" (id 5) (at 135.89 36.83 0)
       (effects (font (size 1.27 1.27)) hide)
     )
@@
       (effects (font (size 1.27 1.27)) hide)
     )
+    (property "LCSC Part" "C25803" (id 5) (at 105.41 72.39 0)
+      (effects (font (size 1.27 1.27)) hide)
+    )
     (pin "1")
     (pin "2")
@@
       (effects (font (size 1.27 1.27)) hide)
     )
+    (property "LCSC Part" "C15849" (id 5) (at 96.52 69.85 0)
+      (effects (font (size 1.27 1.27)) hide)
+    )
     (pin "1")
     (pin "2")
@@
       (effects (font (size 1.27 1.27)) hide)
     )
+    (property "LCSC Part" "C307331" (id 5) (at 139.7 59.69 0)
+      (effects (font (size 1.27 1.27)) hide)
+    )
     (pin "1")
     (pin "2")
@@
       (effects (font (size 1.27 1.27)) hide)
     )
+    (property "LCSC Part" "C408412" (id 5) (at 144.78 67.31 0)
+      (effects (font (size 1.27 1.27)) hide)
+    )
     (pin "1")
     (pin "2")
@@
       (effects (font (size 1.27 1.27)) hide)
     )
+    (property "LCSC Part" "C14663" (id 5) (at 139.7 96.52 0)
+      (effects (font (size 1.27 1.27)) hide)
+    )
     (pin "1")
     (pin "2")
@@
       (effects (font (size 1.27 1.27)) hide)
     )
+    (property "LCSC Part" "C23254" (id 5) (at 143.51 85.09 0)
+      (effects (font (size 1.27 1.27)) hide)
+    )
     (pin "1")
     (pin "2")
@@
     )
     (property "LCSC Part #" "C19666" (id 4) (at 147.32 80.01 0)
+      (effects (font (size 1.27 1.27)) hide)
+    )
+    (property "LCSC Part" "C19666" (id 5) (at 147.32 80.01 0)
       (effects (font (size 1.27 1.27)) hide)
     )
@@
       (effects (font (size 1.27 1.27)) hide)
     )
+    (property "LCSC Part" "C23231" (id 5) (at 152.4 69.85 0)
+      (effects (font (size 1.27 1.27)) hide)
+    )
     (pin "1")
     (pin "2")
@@
       (effects (font (size 1.27 1.27)) hide)
     )
+    (property "LCSC Part" "C22797" (id 5) (at 152.4 76.2 0)
+      (effects (font (size 1.27 1.27)) hide)
+    )
     (pin "1")
     (pin "2")
@@
     )
     (property "LCSC Part #" "C1634" (id 4) (at 156.21 69.85 0)
+      (effects (font (size 1.27 1.27)) hide)
+    )
+    (property "LCSC Part" "C1634" (id 5) (at 156.21 69.85 0)
       (effects (font (size 1.27 1.27)) hide)
     )
@@
       (effects (font (size 1.27 1.27)) hide)
     )
+    (property "LCSC Part" "C22859" (id 5) (at 162.56 80.01 0)
+      (effects (font (size 1.27 1.27)) hide)
+    )
     (pin "1")
     (pin "2")
@@
       (effects (font (size 1.27 1.27)) hide)
     )
+    (property "LCSC Part" "C12891" (id 5) (at 166.37 69.85 0)
+      (effects (font (size 1.27 1.27)) hide)
+    )
     (pin "1")
     (pin "2")
@@
     )
     (property "LCSC Part #" "C12891" (id 4) (at 173.99 69.85 0)
+      (effects (font (size 1.27 1.27)) hide)
+    )
+    (property "LCSC Part" "C12891" (id 5) (at 173.99 69.85 0)
       (effects (font (size 1.27 1.27)) hide)
     )
@@
     )
     (property "Datasheet" "~" (id 3) (at 223.52 78.74 0)
+      (effects (font (size 1.27 1.27)) hide)
+    )
+    (property "JLCPCB BOM" "0" (id 4) (at 223.52 78.74 0)
       (effects (font (size 1.27 1.27)) hide)
     )
@@
       (effects (font (size 1.27 1.27)) hide)
     )
+    (property "LCSC Part" "C7950" (id 5) (at 41.91 167.64 0)
+      (effects (font (size 1.27 1.27)) hide)
+    )
     (pin "1")
     (pin "2")
@@
     )
     (property "LCSC Part #" "C23253" (id 4) (at 144.78 172.72 0)
+      (effects (font (size 1.27 1.27)) hide)
+    )
+    (property "LCSC Part" "C23253" (id 5) (at 144.78 172.72 0)
       (effects (font (size 1.27 1.27)) hide)
     )
@@
     )
     (property "LCSC Part #" "C7950" (id 4) (at 76.2 167.64 0)
+      (effects (font (size 1.27 1.27)) hide)
+    )
+    (property "LCSC Part" "C7950" (id 5) (at 76.2 167.64 0)
       (effects (font (size 1.27 1.27)) hide)
     )
@@
       (effects (font (size 1.27 1.27)) hide)
     )
+    (property "JLCPCB BOM" "0" (id 4) (at 128.27 120.65 0)
+      (effects (font (size 1.27 1.27)) hide)
+    )
     (pin "1")
     (pin "2")
@@
       (effects (font (size 1.27 1.27)) hide)
     )
+    (property "LCSC Part" "C72041" (id 5) (at 144.78 165.1 0)
+      (effects (font (size 1.27 1.27)) hide)
+    )
     (pin "1")
     (pin "2")
@@
     )
     (property "LCSC Part #" "C15127" (id 4) (at 57.15 167.64 0)
+      (effects (font (size 1.27 1.27)) hide)
+    )
+    (property "LCSC Part" "C15127" (id 5) (at 57.15 167.64 0)
       (effects (font (size 1.27 1.27)) hide)
     )
@@
       (effects (font (size 1.27 1.27)) hide)
     )
+    (property "LCSC Part" "C15127" (id 5) (at 44.45 78.74 0)
+      (effects (font (size 1.27 1.27)) hide)
+    )
     (pin "1")
     (pin "2")
@@
     )
     (property "Datasheet" "~" (id 3) (at 49.53 53.34 0)
+      (effects (font (size 1.27 1.27)) hide)
+    )
+    (property "JLCPCB BOM" "0" (id 4) (at 49.53 53.34 0)
       (effects (font (size 1.27 1.27)) hide)
     )
@@
       (effects (font (size 1.27 1.27)) hide)
     )
+    (property "JLCPCB BOM" "0" (id 4) (at 34.29 104.14 0)
+      (effects (font (size 1.27 1.27)) hide)
+    )
     (pin "1")
     (pin "2")
@@
     )
     (property "Datasheet" "~" (id 3) (at 256.54 63.5 0)
+      (effects (font (size 1.27 1.27)) hide)
+    )
+    (property "JLCPCB BOM" "0" (id 4) (at 256.54 63.5 0)
       (effects (font (size 1.27 1.27)) hide)
     )
@@
     )
     (property "Datasheet" "~" (id 3) (at 238.76 115.57 0)
+      (effects (font (size 1.27 1.27)) hide)
+    )
+    (property "JLCPCB BOM" "0" (id 4) (at 238.76 115.57 0)
       (effects (font (size 1.27 1.27)) hide)
     )
@@
       (effects (font (size 1.27 1.27)) hide)
     )
+    (property "JLCPCB BOM" "0" (id 4) (at 256.54 76.2 0)
+      (effects (font (size 1.27 1.27)) hide)
+    )
     (pin "1")
     (pin "2")
@@
     )
     (property "Datasheet" "~" (id 3) (at 39.37 54.61 0)
+      (effects (font (size 1.27 1.27)) hide)
+    )
+    (property "JLCPCB BOM" "0" (id 4) (at 35.56 53.34 0)
       (effects (font (size 1.27 1.27)) hide)
     )
@@
       (effects (font (size 1.27 1.27)) hide)
     )
+    (property "JLCPCB BOM" "0" (id 4) (at 40.64 123.19 0)
+      (effects (font (size 1.27 1.27)) hide)
+    )
     (pin "1")
     (pin "2")
@@
     )
     (property "Datasheet" "~" (id 3) (at 241.3 99.06 0)
+      (effects (font (size 1.27 1.27)) hide)
+    )
+    (property "JLCPCB BOM" "0" (id 4) (at 241.3 99.06 0)
       (effects (font (size 1.27 1.27)) hide)
     )
@@
       (effects (font (size 1.27 1.27)) hide)
     )
+    (property "LCSC Part" "C25077" (id 5) (at 130.81 55.88 0)
+      (effects (font (size 1.27 1.27)) hide)
+    )
     (pin "1")
     (pin "2")
@@
       (effects (font (size 1.27 1.27)) hide)
     )
+    (property "LCSC Part" "C23630" (id 5) (at 116.84 124.46 0)
+      (effects (font (size 1.27 1.27)) hide)
+    )
     (pin "1")
     (pin "2")
@@
     )
     (property "Datasheet" "" (id 3) (at 123.19 74.93 0)
+      (effects (font (size 1.27 1.27)) hide)
+    )
+    (property "JLCPCB BOM" "0" (id 4) (at 123.19 74.93 0)
       (effects (font (size 1.27 1.27)) hide)
     )
@@
       (effects (font (size 1.27 1.27)) hide)
     )
+    (property "LCSC Part" "C25819" (id 5) (at 44.45 88.9 0)
+      (effects (font (size 1.27 1.27)) hide)
+    )
     (pin "1")
     (pin "2")
@@
       (effects (font (size 1.27 1.27)) hide)
     )
+    (property "LCSC Part" "C31850" (id 5) (at 26.67 168.91 0)
+      (effects (font (size 1.27 1.27)) hide)
+    )
     (pin "1")
     (pin "2")
@@
       (effects (font (size 1.27 1.27)) hide)
     )
+    (property "LCSC Part" "C7950" (id 5) (at 90.17 168.91 0)
+      (effects (font (size 1.27 1.27)) hide)
+    )
     (pin "5")
     (pin "6")
@@
       (effects (font (size 1.27 1.27)) hide)
     )
+    (property "LCSC Part" "C8678" (id 5) (at 49.53 101.6 0)
+      (effects (font (size 1.27 1.27)) hide)
+    )
     (pin "1")
     (pin "2")
@@
     )
     (property "LCSC Part #" "C1779" (id 4) (at 139.7 124.46 0)
+      (effects (font (size 1.27 1.27)) hide)
+    )
+    (property "LCSC Part" "C1779" (id 5) (at 139.7 124.46 0)
       (effects (font (size 1.27 1.27)) hide)
     )
@@
       (effects (font (size 1.27 1.27)) hide)
     )
+    (property "JLCPCB BOM" "0" (id 4) (at 223.52 62.23 0)
+      (effects (font (size 1.27 1.27)) hide)
+    )
     (pin "1")
     (pin "2")
@@
     )
     (property "Datasheet" "~" (id 3) (at 52.07 81.28 90)
+      (effects (font (size 1.27 1.27)) hide)
+    )
+    (property "JLCPCB BOM" "0" (id 4) (at 52.07 81.28 0)
       (effects (font (size 1.27 1.27)) hide)
     )
@@
       (effects (font (size 1.27 1.27)) hide)
     )
+    (property "LCSC Part" "C23189" (id 5) (at 26.67 161.29 0)
+      (effects (font (size 1.27 1.27)) hide)
+    )
